File: hardware/layout/poc/main/main.kicad_pcb (KiCad board)
At the start: 4 copper layers, 49.5 x 76.5 mm, 71 parts, among them J1 KNX bus terminal pins, J2 AUX, J3 DALI, J4 JST-SH 1x10, Q1 MJD45H11, Q2 BC857, Q3 IRLML0060, Q4 BC847, Q5 BC847, Q6 BC847, U1 NCN5130MNTWG, U2 SCT2400TVBR, U3 REM3-2415S/A 24V->15V 3W iso, U4 TLP383(D4BLLTL,E, U5 TLP383(D4BLLTL,E, U6 LM66100, U7 XIAO ESP32C6, Y1 16MHz

Commit message: CI matrix for hardware variants (poc/v2); updated AGENTS.md with V2 details and verification workflow
Parts:
- moved U5 2.18 mm to (12.0, -43.0)
- moved U4 1.15 mm to (4.50, -43.0)
Routing:
- net KNX_TXD: track 50.5 -> 21.3 mm
- net +5V_XIAO: track 8.09 -> 26.3 mm
- net +5V: track 47.9 -> 37.4 mm, vias 4 -> 2
- net +3V3: track 54.2 -> 63.8 mm, vias 3 -> 4
- net LED_DATA: track 55.3 -> 64.2 mm
- net DALI_RX: track 24.8 -> 33.5 mm
- net VFILT: track 56.3 -> 63.2 mm, vias 3 -> 2
- net N$6: track 25.2 -> 18.7 mm
- net RX_LIM_IN: track 10.4 -> 16.1 mm
- net DALI_SENSE: track 16.7 -> 11.2 mm, vias 2 -> 0
- net N$9: track 4.14 -> 9.24 mm, vias 1 -> 2
- net DALI_GATE_SW: track 25.4 -> 20.9 mm
- net NCN_SAVEB: track 31.7 -> 27.4 mm, vias 2 -> 1
- net LED_DALI: track 40.7 -> 44.2 mm
- net DALI_ISO15V: track 34.2 -> 37.2 mm, vias 1 -> 2
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Other:
- outline, holes or cut-outs redrawn
