File: hardware/layout/v1/main/main.kicad_pcb (KiCad board)
At the start: 4 copper layers, 49.5 x 76.5 mm, 75 parts, among them J1 KNX bus terminal pins, J2 AUX, J3 DALI, J4 JST-SH 1x10, Q1 MJD45H11, Q2 BC857, Q3 IRLML0060, Q4 BC847, Q5 BC847, Q6 BC847, U1 NCN5130MNTWG, U2 SCT2400TVBR, U3 REM3-2415S/A/CTRL 24V->15V 3W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, U4 TLP383, U5 TLP383(D4BLLTL,E, U6 TLP383(D4BLLTL,E, U7 LM66100, U8 XIAO ESP32C6, Y1 16MHz

Commit message: Updated DALI DC-DC converter from RECOM REM3-2415S/A to REC3-2415SRW/H2/A series across all variants, changed V3 OLED from 14-pin 0.5mm ZIF to 14-pin 0.62mm solder-tail FPC connector, and expanded assembly documentation with Mouser/Digi-Key/TME part numbers and alternative suppliers
Parts:
- U3: value REM3-2415S/A/CTRL 24V->15V 3W iso -> REC3-2415SRW/H2/A/CTRL 24V->15V 3W iso
