File: hardware/layout/v2/interface/interface.kicad_pcb (KiCad board)
At the start: 4 copper layers, 31.5 x 27.5 mm, 22 parts, among them J1 Main logic, J2 Main DALI, Q1 IRLML0060, Q2 BC847, Q3 BC847, Q4 BC847, U1 TLP383(D4BLLTL,E, U2 TLP383(D4BLLTL,E

Commit message: Removed V1 hardware variant from CI workflows, updated AGENTS.md documentation to reflect V2/V3-only support
Parts:
- R3: value 22k -> 4k7
- R4: value 100k -> 10k
- R5: value 3R3 -> 2R
- R8: value 10k -> 4k7
