File: hardware/layout/v2/ui/ui.kicad_pcb (KiCad board)
At the start: 4 copper layers, 31.5 x 40.5 mm, 23 parts, among them J1 Controller cable, J2 OLED, SW1 PRG/RST, SW2 FUNC, U1 LM66100, U2 XIAO ESP32C6, U3 74AHCT1G125

Commit message: Removed V1 hardware variant from CI workflows, updated AGENTS.md documentation to reflect V2/V3-only support
Connections:
- U1 pad 3: GND -> +5V_XIAO
Routing:
- net GND: track 128.7 -> 116.0 mm
- net DALI_SUPPLY_OFF: track 40.4 -> 35.0 mm
- net BTN_LADDER: track 56.7 -> 51.6 mm
- net I2C_SCL: track 21.2 -> 25.4 mm
- net +5V_XIAO: track 25.6 -> 29.8 mm
- net N$2: track 21.5 -> 25.0 mm
- net KNX_RXD: track 49.2 -> 46.2 mm
- net I2C_SDA: track 23.2 -> 20.5 mm
- net N$4: track 30.1 -> 32.5 mm
- net +5V: track 69.8 -> 71.9 mm
- net +3V3: track 54.6 -> 56.6 mm
- net N$1: track 16.6 -> 17.5 mm, vias 0 -> 2
- net N$3: track 12.0 -> 12.4 mm, vias 0 -> 2

Commit message: Unified V2/V3 UI buttons to Omron B3U-1000P with cover spring tabs
Parts:
- SW1, SW2: footprint Button_Switch_SMD:SW_SPST_PTS645Sx43SMTR92 -> Button_Switch_SMD:SW_SPST_B3U-1000P
- turned SW1 to 90 degrees
- turned SW2 to 90 degrees
Routing:
- net N$1: track 17.5 -> 8.32 mm
- net N$2: track 25.0 -> 16.0 mm
- net BTN_LADDER: track 51.6 -> 44.6 mm, vias 2 -> 3
- net GND: track 116.0 -> 122.6 mm, vias 1 -> 2
- net +3V3: track 56.6 -> 61.8 mm
- net +5V_XIAO: track 29.8 -> 25.4 mm
- net +5V: track 71.9 -> 68.2 mm
- net I2C_SDA: track 20.5 -> 23.5 mm
- net KNX_RXD: track 46.2 -> 43.5 mm
- net I2C_SCL: track 25.4 -> 23.1 mm
- net N$4: track 32.5 -> 30.5 mm
- net DALI_SUPPLY_OFF: track 35.0 -> 36.4 mm
- net KNX_TXD: track 31.7 -> 32.7 mm
